File: hardware/atmega168_tb2.kicad_pcb (KiCad board)
At the start: 2 copper layers, 80 x 30 mm, 23 parts, among them J1 AVR-ISP-6, J2 WAVESHARE, J3 DBG_CARD, J4 Micro_SD_Card_Det, J5 BATT, J6 RX, J7 PE0, J8 PE1, J9 GND, Q1 P_FET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

Commit message: updated kicad hardware project
Other:
- net class Default removed
