File: hardware/atmega168_tb2.kicad_sch (KiCad schematic)
At the start: 23 parts, among them J1 AVR-ISP-6, J2 WAVESHARE, J3 DBG_CARD, J4 Micro_SD_Card_Det, J5 BATT, J6 RX, J7 PE0, J8 PE1, J9 GND, Q1 P_FET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

Commit message: got serial output of avr to work
Connections:
- net PPWRCTRL: no longer U2.11 (PD7)
- net P_BUSY: now also U2.11 (PD7); no longer U2.31 (PD1)
Changed lines of the file:
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@@
     )
   )
-  (global_label "P_BUSY" (shape input) (at 105.41 90.17 0)
+  (global_label "P_BUSY" (shape input) (at 105.41 105.41 0)
     (effects (font (size 1.27 1.27)) (justify left))
-    (property "Intersheetrefs" "${INTERSHEET_REFS}" (at 105.41 90.17 0)
+    (property "Intersheetrefs" "${INTERSHEET_REFS}" (at 105.41 105.41 0)
       (effects (font (size 1.27 1.27)) hide)
     )
@@
     )
   )
-  (global_label "PPWRCTRL" (shape input) (at 105.41 105.41 0)
+  (global_label "PPWRCTRL" (shape input) (at 110.49 107.95 0)
     (effects (font (size 1.27 1.27)) (justify left))
-    (property "Intersheetrefs" "${INTERSHEET_REFS}" (at 105.41 105.41 0)
+    (property "Intersheetrefs" "${INTERSHEET_REFS}" (at 110.49 107.95 0)
       (effects (font (size 1.27 1.27)) hide)
     )
